File: ppm.kicad_pcb (KiCad board)
At the start: 2 copper layers, 40 x 50 mm, 28 parts, among them J1 Conn_01x04, J2 Conn_01x04, J3 Conn_01x03, J4 Conn_01x06, SW1 PC0, SW2 PC1, SW3 PC2, U1 ATmega48-20AU, U2 KA78M05_TO252

Commit message: done
Parts:
- removed the REF** at (23.7, 66.6)
- removed the REF** at (56.4, 66.6)
- removed the REF** at (23.6, 23.7)
- removed the REF** at (56.2, 23.7)
- added REF**: MountingHole_2.5mm, MountingHole:MountingHole_2.5mm, F.Cu at (24.0, 65.5)
- added REF**: MountingHole_2.5mm, MountingHole:MountingHole_2.5mm, F.Cu at (55.9, 24.2)
- added REF**: MountingHole_2.5mm, MountingHole:MountingHole_2.5mm, F.Cu at (23.9, 23.9)
- SW1: value PC0 -> PC2
- SW3: value PC2 -> PC0
- moved R3 37.2 mm to (26.4, 33.7), turned to 90 degrees
- moved R4 36.1 mm to (26.4, 37.9), turned to 90 degrees
- moved J4 35.9 mm to (57.6, 35.8), turned to 270 degrees
- moved R7 16.6 mm to (46.3, 54.5)
- moved SW3 16.6 mm to (53.6, 54.5)
- moved R6 15.1 mm to (46.3, 59.7)
- moved SW2 15.1 mm to (53.6, 59.7)
- moved R5 13.6 mm to (46.3, 64.9)
- moved SW1 13.6 mm to (53.6, 64.9)
- moved D3 11.6 mm to (32.0, 64.8), turned to 270 degrees
- moved U1 11.1 mm to (45.4, 39.4), turned to 270 degrees
- moved R11 8.93 mm to (32.0, 59.5), turned to 270 degrees
- moved D2 8.09 mm to (36.0, 64.8), turned to 270 degrees
- moved D1 7.86 mm to (40.1, 64.8), turned to 270 degrees
- moved C1 4.88 mm to (44.5, 48.0), turned to 0 degrees
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Connections:
- J4 pad 3: /mosi -> /rst
- J4 pad 4: /rst -> /sck
- J4 pad 5: /sck -> /miso
- J4 pad 6: /miso -> /mosi
- R5 pad 2: /PC0 -> /PC2
- R7 pad 2: /PC2 -> /PC0
- SW1 pad 1: /PC0 -> /PC2
- SW3 pad 1: /PC2 -> /PC0
- U1 pad 1: Net-(U1-Pad1) -> (no net)
- U1 pad 10: Net-(U1-Pad10) -> (no net)
- U1 pad 11: Net-(U1-Pad11) -> (no net)
- U1 pad 12: /led1 -> /led3
- U1 pad 14: /led3 -> /led1
- U1 pad 19: Net-(U1-Pad19) -> (no net)
- U1 pad 2: Net-(U1-Pad2) -> (no net)
- U1 pad 22: Net-(U1-Pad22) -> (no net)
- U1 pad 26: Net-(U1-Pad26) -> /PC3
- U1 pad 32: Net-(U1-Pad32) -> (no net)
- U1 pad 7: Net-(U1-Pad7) -> (no net)
- U1 pad 8: Net-(U1-Pad8) -> (no net)
- U1 pad 9: Net-(U1-Pad9) -> (no net)
Routing:
- net +5V: track 82.0 -> 155.5 mm, vias 2 -> 0
- net /led3: track 8.29 -> 32.1 mm
- net /PC3: track 13.4 -> 33.9 mm, vias 0 -> 2
- net /rst: track 28.8 -> 9.80 mm, vias 1 -> 0
- net /SCL: track 14.3 -> 31.3 mm, vias 0 -> 1
- net /SDA: track 16.8 -> 33.2 mm, vias 0 -> 1
- net /led2: track 13.5 -> 29.6 mm
- net /PC2: track 12.1 -> 26.6 mm
- net /led1: track 17.5 -> 30.1 mm
- net GND: track 30.5 -> 19.0 mm, vias 14 -> 16
- net /RXD: track 33.5 -> 43.7 mm, vias 0 -> 1
- net /PC1: track 12.5 -> 20.1 mm
- net /TXD: track 34.4 -> 40.8 mm, vias 0 -> 1
- net /PC0: track 18.5 -> 13.5 mm
- net /mosi: track 20.8 -> 18.7 mm
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Other:
- board text added: "MOSI | MISO | SCK | RST | GND | 5V"
- board text removed: "MISO | SCK | RST | MOSI | GND | 5V"
